File: hardware/riscv_pc/power.kicad_sch (KiCad schematic)
At the start: 7 parts, among them CN1 S2B-PH-SM4-TB(LF)(SN), SW2 SS11-BBIWJ-R20-R, U1 TP4056_BREAKOUT, U3 TPS61027DRCR

Commit message: Create PCB
Parts:
- removed C3: 100u, Capacitor_SMD:CP_Elec_6.3x7.7, symbol Device:C_Polarized
- removed C4: 10uF, symbol Device:C
- added C?: UWX1C101MCL1GB, easyeda2kicad:CAP-SMD_BD6.3-L6.6-W6.6-FD, symbol lcsc:UWX1C101MCL1GB
- added C?: CL31A106KBHNNNE, easyeda2kicad:C1206, symbol lcsc:CL31A106KBHNNNE
Connections:
- net +5V: now also C?.1
- net BAT+: now also C?.2
- net GND: now also C?.1, C?.2
Changed lines of the file:
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@@
     (pin "1")
   )
-  (symbol (lib_id "Device:C") (at 153.67 62.738 270) (unit 1)
-    (in_bom yes) (on_board yes)
-    (property "Reference" "C4" (id 0) (at 154.94 66.548 90)
-      (effects (font (size 1.27 1.27)) (justify right))
-    )
-    (property "Value" "10uF" (id 1) (at 156.21 58.928 90)
-      (effects (font (size 1.27 1.27)) (justify right))
-    )
-    (property "Footprint" "" (id 2) (at 149.86 63.7032 0)
-      (effects (font (size 1.27 1.27)) hide)
-    )
-    (property "Datasheet" "~" (id 3) (at 153.67 62.738 0)
+  (symbol (lib_id "lcsc:UWX1C101MCL1GB") (at 41.91 102.87 270) (unit 1)
+    (in_bom yes) (on_board yes)
+    (property "Reference" "C?" (id 0) (at 44.704 102.87 90)
+      (effects (font (size 1.27 1.27)) (justify left))
+    )
+    (property "Value" "UWX1C101MCL1GB" (id 1) (at 45.72 103.5349 90)
+      (effects (font (size 1.27 1.27)) (justify left) hide)
+    )
+    (property "Footprint" "easyeda2kicad:CAP-SMD_BD6.3-L6.6-W6.6-FD" (id 2) (at 34.29 102.87 0)
+      (effects (font (size 1.27 1.27)) hide)
+    )
+    (property "Datasheet" "https://lcsc.com/product-detail/Aluminum-Electrolytic-Capacitors-SMD_Nichicon_UWX1C101MCL1GB_100uF-16V-20_C111600.html" (id 3) (at 31.75 102.87 0)
+      (effects (font (size 1.27 1.27)) hide)
+    )
+    (property "Manufacturer" "Nichicon(尼吉康)" (id 4) (at 29.21 102.87 0)
+      (effects (font (size 1.27 1.27)) hide)
+    )
+    (property "LCSC Part" "C111600" (id 5) (at 26.67 102.87 0)
+      (effects (font (size 1.27 1.27)) hide)
+    )
+    (property "JLC Part" "Extended Part" (id 6) (at 24.13 102.87 0)
       (effects (font (size 1.27 1.27)) hide)
     )
@@
     )
     (pin "1")
+  )
+  (symbol (lib_id "lcsc:CL31A106KBHNNNE") (at 153.67 62.738 0) (unit 1)
+    (in_bom yes) (on_board yes)
+    (property "Reference" "C?" (id 0) (at 153.67 59.182 0))
+    (property "Value" "CL31A106KBHNNNE" (id 1) (at 153.67 66.548 0)
+      (effects (font (size 1.27 1.27)) hide)
+    )
+    (property "Footprint" "easyeda2kicad:C1206" (id 2) (at 153.67 70.358 0)
+      (effects (font (size 1.27 1.27)) hide)
+    )
+    (property "Datasheet" "https://lcsc.com/product-detail/Multilayer-Ceramic-Capacitors-MLCC-SMD-SMT_SAMSUNG_CL31A106KBHNNNE_10uF-106-10-50V_C13585.html" (id 3) (at 153.67 72.898 0)
+      (effects (font (size 1.27 1.27)) hide)
+    )
+    (property "Manufacturer" "SAMSUNG(三星)" (id 4) (at 153.67 75.438 0)
+      (effects (font (size 1.27 1.27)) hide)
+    )
+    (property "LCSC Part" "C13585" (id 5) (at 153.67 77.978 0)
+      (effects (font (size 1.27 1.27)) hide)
+    )
+    (property "JLC Part" "Basic Part" (id 6) (at 153.67 80.518 0)
+      (effects (font (size 1.27 1.27)) hide)
+    )
+    (pin "1")
+    (pin "2")
   )
   (symbol (lib_id "lcsc:SM7850-6R8MT") (at 177.8 62.738 0) (unit 1)
@@
     (pin "1")
   )
-  (symbol (lib_id "Device:C_Polarized") (at 41.91 102.87 0) (unit 1)
-    (in_bom yes) (on_board yes) (fields_autoplaced)
-    (property "Reference" "C3" (id 0) (at 44.831 101.0725 0)
-      (effects (font (size 1.27 1.27)) (justify left))
-    )
-    (property "Value" "100u" (id 1) (at 44.831 103.8476 0)
-      (effects (font (size 1.27 1.27)) (justify left))
-    )
-    (property "Footprint" "Capacitor_SMD:CP_Elec_6.3x7.7" (id 2) (at 42.8752 106.68 0)
-      (effects (font (size 1.27 1.27)) hide)
-    )
-    (property "Datasheet" "~" (id 3) (at 41.91 102.87 0)
-      (effects (font (size 1.27 1.27)) hide)
-    )
-    (pin "1")
-    (pin "2")
-  )
   (symbol (lib_id "power:GND") (at 171.45 50.038 90) (unit 1)
