File: hardware/riscv_pc/riscv_pc.kicad_sch (KiCad schematic)
At the start: 16 parts, among them J1 te_m.2_b, J2 te_m.2_b, J4 HDMI_A, J5 AudioJack3, SW1 TS-1187A-C-D-B

Commit message: Create PCB
Parts:
- removed C1, C2: 10u, Capacitor_SMD:C_0603_1608Metric, symbol Device:C
- added C? (x2): CL31A106KBHNNNE, easyeda2kicad:C1206, symbol lcsc:CL31A106KBHNNNE
Connections:
- net HP_LEFT: now also C?.2
- net HP_RIGHT: now also C?.1
- net at D11.1 (K), J5.T: now also C?.2
- net at D10.1 (K), J5.R: now also C?.1
Changed lines of the file:
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@@
     (pin "9")
+  )
+  (symbol (lib_id "lcsc:CL31A106KBHNNNE") (at 142.24 46.228 90) (unit 1)
+    (in_bom yes) (on_board yes)
+    (property "Reference" "C?" (id 0) (at 137.16 46.228 90)
+      (effects (font (size 1.27 1.27)) (justify right))
+    )
+    (property "Value" "CL31A106KBHNNNE" (id 1) (at 146.05 47.4979 90)
+      (effects (font (size 1.27 1.27)) (justify right) hide)
+    )
+    (property "Footprint" "easyeda2kicad:C1206" (id 2) (at 149.86 46.228 0)
+      (effects (font (size 1.27 1.27)) hide)
+    )
+    (property "Datasheet" "https://lcsc.com/product-detail/Multilayer-Ceramic-Capacitors-MLCC-SMD-SMT_SAMSUNG_CL31A106KBHNNNE_10uF-106-10-50V_C13585.html" (id 3) (at 152.4 46.228 0)
+      (effects (font (size 1.27 1.27)) hide)
+    )
+    (property "Manufacturer" "SAMSUNG(三星)" (id 4) (at 154.94 46.228 0)
+      (effects (font (size 1.27 1.27)) hide)
+    )
+    (property "LCSC Part" "C13585" (id 5) (at 157.48 46.228 0)
+      (effects (font (size 1.27 1.27)) hide)
+    )
+    (property "JLC Part" "Basic Part" (id 6) (at 160.02 46.228 0)
+      (effects (font (size 1.27 1.27)) hide)
+    )
+    (pin "1")
+    (pin "2")
   )
   (symbol (lib_name "GND_5") (lib_id "power:GND") (at 226.06 156.464 0) (unit 1)
@@
     (pin "1")
   )
+  (symbol (lib_id "lcsc:CL31A106KBHNNNE") (at 150.368 52.578 0) (unit 1)
+    (in_bom yes) (on_board yes)
+    (property "Reference" "C?" (id 0) (at 150.368 49.53 0))
+    (property "Value" "CL31A106KBHNNNE" (id 1) (at 150.622 55.626 0)
+      (effects (font (size 1.27 1.27)) hide)
+    )
+    (property "Footprint" "easyeda2kicad:C1206" (id 2) (at 150.368 60.198 0)
+      (effects (font (size 1.27 1.27)) hide)
+    )
+    (property "Datasheet" "https://lcsc.com/product-detail/Multilayer-Ceramic-Capacitors-MLCC-SMD-SMT_SAMSUNG_CL31A106KBHNNNE_10uF-106-10-50V_C13585.html" (id 3) (at 150.368 62.738 0)
+      (effects (font (size 1.27 1.27)) hide)
+    )
+    (property "Manufacturer" "SAMSUNG(三星)" (id 4) (at 150.368 65.278 0)
+      (effects (font (size 1.27 1.27)) hide)
+    )
+    (property "LCSC Part" "C13585" (id 5) (at 150.368 67.818 0)
+      (effects (font (size 1.27 1.27)) hide)
+    )
+    (property "JLC Part" "Basic Part" (id 6) (at 150.368 70.358 0)
+      (effects (font (size 1.27 1.27)) hide)
+    )
+    (pin "1")
+    (pin "2")
+  )
   (symbol (lib_name "+5V_2") (lib_id "power:+5V") (at 233.68 116.078 0) (unit 1)
     (in_bom yes) (on_board yes)
@@
     (pin "1")
   )
-  (symbol (lib_id "Device:C") (at 142.24 46.228 0) (unit 1)
-    (in_bom yes) (on_board yes)
-    (property "Reference" "C1" (id 0) (at 137.668 44.196 0)
-      (effects (font (size 1.27 1.27)) (justify left))
-    )
-    (property "Value" "10u" (id 1) (at 137.16 48.26 0)
-      (effects (font (size 1.27 1.27)) (justify left))
-    )
-    (property "Footprint" "Capacitor_SMD:C_0603_1608Metric" (id 2) (at 143.2052 50.038 0)
-      (effects (font (size 1.27 1.27)) hide)
-    )
-    (property "Datasheet" "~" (id 3) (at 142.24 46.228 0)
-      (effects (font (size 1.27 1.27)) hide)
-    )
-    (property "JLC" "C96446" (id 4) (at 142.24 46.228 0)
-      (effects (font (size 1.27 1.27)) hide)
-    )
-    (property "LCSC" "C96446" (id 5) (at 142.24 46.228 0)
-      (effects (font (size 1.27 1.27)) hide)
-    )
-    (pin "1")
-    (pin "2")
-  )
   (symbol (lib_name "GND_1") (lib_id "power:GND") (at 149.606 27.432 0) (unit 1)
     (in_bom yes) (on_board yes)
@@
     (pin "4")
   )
-  (symbol (lib_id "Device:C") (at 150.368 52.578 90) (unit 1)
-    (in_bom yes) (on_board yes) (fields_autoplaced)
-    (property "Reference" "C2" (id 0) (at 150.368 46.4525 90))
-    (property "Value" "10u" (id 1) (at 150.368 49.2276 90))
-    (property "Footprint" "Capacitor_SMD:C_0603_1608Metric" (id 2) (at 154.178 51.6128 0)
-      (effects (font (size 1.27 1.27)) hide)
-    )
-    (property "Datasheet" "~" (id 3) (at 150.368 52.578 0)
-      (effects (font (size 1.27 1.27)) hide)
-    )
-    (property "JLC" "C96446" (id 4) (at 150.368 52.578 0)
-      (effects (font (size 1.27 1.27)) hide)
-    )
-    (property "LCSC" "C96446" (id 5) (at 150.368 52.578 0)
-      (effects (font (size 1.27 1.27)) hide)
-    )
-    (pin "1")
-    (pin "2")
-  )
   (symbol (lib_id "Device:R") (at 95.82 176.25 90) (unit 1)
     (in_bom yes) (on_board yes) (fields_autoplaced)
@@
       (reference "#PWR0132") (unit 1) (value "GND") (footprint "")
     )
-    (path "/a1b6a1f7-8cfa-4da6-90b7-efbdfe57a4c1"
-      (reference "C1") (unit 1) (value "10u") (footprint "Capacitor_SMD:C_0603_1608Metric")
-    )
-    (path "/d955015d-c318-41a0-a394-a8fb19bd8eee"
-      (reference "C2") (unit 1) (value "10u") (footprint "Capacitor_SMD:C_0603_1608Metric")
-    )
-    (path "/561ad5b5-1f0b-46c2-8c8e-c222b229715f/e8ef0fdd-bf38-4075-875d-877a5ddc449b"
-      (reference "C3") (unit 1) (value "100u") (footprint "Capacitor_SMD:CP_Elec_6.3x7.7")
-    )
-    (path "/561ad5b5-1f0b-46c2-8c8e-c222b229715f/2ec57f63-8459-43c5-8ce4-f76f22057b57"
-      (reference "C4") (unit 1) (value "10uF") (footprint "")
-    )
-    (path "/16053816-87f9-4442-aa90-5aa52c7c4ff8/87d18a6c-c8b6-427e-97f8-654a65309b20"
-      (reference "C5") (unit 1) (value "10uF") (footprint "")
-    )
-    (path "/16053816-87f9-4442-aa90-5aa52c7c4ff8/a3b27de0-95e4-4720-9afe-74d1150e92ac"
-      (reference "C6") (unit 1) (value "10uF") (footprint "")
+    (path "/0815db2e-14eb-4028-9b83-0520336546cf"
+      (reference "C?") (unit 1) (value "CL31A106KBHNNNE") (footprint "easyeda2kicad:C1206")
+    )
+    (path "/561ad5b5-1f0b-46c2-8c8e-c222b229715f/2fd049d2-e9b2-46b6-83d9-b8aca04af7c4"
+      (reference "C?") (unit 1) (value "UWX1C101MCL1GB") (footprint "easyeda2kicad:CAP-SMD_BD6.3-L6.6-W6.6-FD")
+    )
+    (path "/68824cda-45ce-4388-9fb3-d7f04c24fc19"
+      (reference "C?") (unit 1) (value "CL31A106KBHNNNE") (footprint "easyeda2kicad:C1206")
+    )
+    (path "/561ad5b5-1f0b-46c2-8c8e-c222b229715f/7752f79f-c02e-48c0-b073-a3d3a189c0c5"
+      (reference "C?") (unit 1) (value "CL31A106KBHNNNE") (footprint "easyeda2kicad:C1206")
+    )
+    (path "/16053816-87f9-4442-aa90-5aa52c7c4ff8/b8099d40-6cd5-4f34-9848-fb1c98ff631a"
+      (reference "C?") (unit 1) (value "CL31A106KBHNNNE") (footprint "easyeda2kicad:C1206")
+    )
+    (path "/16053816-87f9-4442-aa90-5aa52c7c4ff8/fc8215b0-ea81-47da-b368-11ff04031fd9"
+      (reference "C?") (unit 1) (value "CL31A106KBHNNNE") (footprint "easyeda2kicad:C1206")
     )
     (path "/561ad5b5-1f0b-46c2-8c8e-c222b229715f/c28cf00c-316b-4f46-9a8c-d59921c06454"
